File: ortho_12x5/ortho_12x5.kicad_pcb (KiCad board)
At the start: 2 copper layers, 120 parts, among them SW1 SW_SPST, SW10 SW_SPST, SW11 SW_SPST, SW12 SW_SPST, SW13 SW_SPST, SW14 SW_SPST, SW15 SW_SPST, SW16 SW_SPST, SW17 SW_SPST, SW18 SW_SPST, SW19 SW_SPST, SW2 SW_SPST, SW20 SW_SPST, SW21 SW_SPST, SW22 SW_SPST, SW23 SW_SPST, SW24 SW_SPST, SW25 SW_SPST, SW26 SW_SPST, SW27 SW_SPST, SW28 SW_SPST, SW29 SW_SPST, SW3 SW_SPST, SW30 SW_SPST, SW31 SW_SPST, SW32 SW_SPST, SW33 SW_SPST, SW34 SW_SPST, SW35 SW_SPST, SW36 SW_SPST, SW37 SW_SPST, SW38 SW_SPST, SW39 SW_SPST, SW4 SW_SPST, SW40 SW_SPST, SW41 SW_SPST, SW42 SW_SPST, SW43 SW_SPST, SW44 SW_SPST, SW45 SW_SPST, SW46 SW_SPST, SW47 SW_SPST, SW48 SW_SPST, SW49 SW_SPST, SW5 SW_SPST, SW50 SW_SPST, SW51 SW_SPST, SW52 SW_SPST, SW53 SW_SPST, SW54 SW_SPST, SW55 SW_SPST, SW56 SW_SPST, SW57 SW_SPST, SW58 SW_SPST, SW59 SW_SPST, SW6 SW_SPST, SW60 SW_SPST, SW7 SW_SPST, SW8 SW_SPST, SW9 SW_SPST

Commit message: Redo schematic
Parts:
- added J1: Conn_01x05, Connector_PinSocket_2.54mm:PinSocket_1x05_P2.54mm_Horizontal, F.Cu at (74.9, -102.9)
- added J2: Conn_01x12, Connector_PinHeader_2.54mm:PinHeader_1x12_P2.54mm_Horizontal, F.Cu at (114.3, 182.9)
- moved D56 189.0 mm to (104.1, 14.0), turned to 0 degrees
- moved D57 188.0 mm to (104.1, 19.1), turned to 0 degrees
- moved D60 187.4 mm to (101.6, 35.6), turned to 0 degrees
- moved D59 187.3 mm to (102.9, 30.5), turned to 0 degrees
- moved D58 187.3 mm to (104.1, 25.4), turned to 0 degrees
- moved D12 180.1 mm to (257.8, 21.6), turned to 0 degrees
- moved D13 178.2 mm to (259.1, 27.9), turned to 0 degrees
- moved D14 174.6 mm to (257.8, 33.0), turned to 0 degrees
- moved D8 167.7 mm to (275.6, 27.9), turned to 0 degrees
- moved D54 165.6 mm to (118.1, 30.5), turned to 0 degrees
- moved D55 165.4 mm to (116.8, 35.6), turned to 0 degrees
- moved D51 164.7 mm to (121.9, 16.5), turned to 0 degrees
- moved D53 164.4 mm to (120.7, 25.4), turned to 0 degrees
- moved D9 164.0 mm to (275.6, 33.0), turned to 0 degrees
- moved D52 163.6 mm to (121.9, 21.6), turned to 0 degrees
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Connections:
- SW1 pad 1: Net-(SW1-Pad1) -> Net-(J1-Pad1)
- SW10 pad 1: Net-(D5-Pad2) -> Net-(J1-Pad5)
- SW11 pad 1: Net-(D6-Pad2) -> Net-(J1-Pad1)
- SW12 pad 1: Net-(D7-Pad2) -> Net-(J1-Pad2)
- SW13 pad 1: Net-(D8-Pad2) -> Net-(J1-Pad3)
- SW14 pad 1: Net-(D9-Pad2) -> Net-(J1-Pad4)
- SW15 pad 1: Net-(D10-Pad2) -> Net-(J1-Pad5)
- SW16 pad 1: Net-(D11-Pad2) -> Net-(J1-Pad1)
- SW17 pad 1: Net-(D12-Pad2) -> Net-(J1-Pad2)
- SW18 pad 1: Net-(D13-Pad2) -> Net-(J1-Pad3)
- SW19 pad 1: Net-(D14-Pad2) -> Net-(J1-Pad4)
- SW2 pad 1: Net-(SW2-Pad1) -> Net-(J1-Pad2)
- SW20 pad 1: Net-(D15-Pad2) -> Net-(J1-Pad5)
- SW21 pad 1: Net-(D16-Pad2) -> Net-(J1-Pad1)
- SW22 pad 1: Net-(D17-Pad2) -> Net-(J1-Pad2)
- SW23 pad 1: Net-(D18-Pad2) -> Net-(J1-Pad3)
- SW24 pad 1: Net-(D19-Pad2) -> Net-(J1-Pad4)
- SW25 pad 1: Net-(D20-Pad2) -> Net-(J1-Pad5)
- SW26 pad 1: Net-(D21-Pad2) -> Net-(J1-Pad1)
- SW27 pad 1: Net-(D22-Pad2) -> Net-(J1-Pad2)
- SW28 pad 1: Net-(D23-Pad2) -> Net-(J1-Pad3)
- SW29 pad 1: Net-(D24-Pad2) -> Net-(J1-Pad4)
- SW3 pad 1: Net-(SW3-Pad1) -> Net-(J1-Pad3)
- SW30 pad 1: Net-(D25-Pad2) -> Net-(J1-Pad5)
- SW31 pad 1: Net-(D26-Pad2) -> Net-(J1-Pad1)
- SW32 pad 1: Net-(D27-Pad2) -> Net-(J1-Pad2)
- SW33 pad 1: Net-(D28-Pad2) -> Net-(J1-Pad3)
- SW34 pad 1: Net-(D29-Pad2) -> Net-(J1-Pad4)
- SW35 pad 1: Net-(D30-Pad2) -> Net-(J1-Pad5)
- SW36 pad 1: Net-(D31-Pad2) -> Net-(J1-Pad1)
- SW37 pad 1: Net-(D32-Pad2) -> Net-(J1-Pad2)
- SW38 pad 1: Net-(D33-Pad2) -> Net-(J1-Pad3)
- SW39 pad 1: Net-(D34-Pad2) -> Net-(J1-Pad4)
- SW4 pad 1: Net-(SW4-Pad1) -> Net-(J1-Pad4)
- SW40 pad 1: Net-(D35-Pad2) -> Net-(J1-Pad5)
- SW41 pad 1: Net-(D36-Pad2) -> Net-(SW41-Pad1)
- SW42 pad 1: Net-(D37-Pad2) -> Net-(SW42-Pad1)
- SW43 pad 1: Net-(D38-Pad2) -> Net-(SW43-Pad1)
- SW44 pad 1: Net-(D39-Pad2) -> Net-(SW44-Pad1)
- SW45 pad 1: Net-(D40-Pad2) -> Net-(SW45-Pad1)
- SW46 pad 1: Net-(D41-Pad2) -> Net-(J1-Pad1)
- SW47 pad 1: Net-(D42-Pad2) -> Net-(J1-Pad2)
- SW48 pad 1: Net-(D43-Pad2) -> Net-(J1-Pad3)
- SW49 pad 1: Net-(D44-Pad2) -> Net-(J1-Pad4)
- SW5 pad 1: Net-(SW5-Pad1) -> Net-(J1-Pad5)
- SW50 pad 1: Net-(D45-Pad2) -> Net-(J1-Pad5)
- SW51 pad 1: Net-(D46-Pad2) -> Net-(J1-Pad1)
- SW52 pad 1: Net-(D47-Pad2) -> Net-(J1-Pad2)
- SW53 pad 1: Net-(D48-Pad2) -> Net-(J1-Pad3)
- SW54 pad 1: Net-(D49-Pad2) -> Net-(J1-Pad4)
- SW55 pad 1: Net-(D50-Pad2) -> Net-(J1-Pad5)
- SW56 pad 1: Net-(D51-Pad2) -> Net-(J1-Pad1)
- SW57 pad 1: Net-(D52-Pad2) -> Net-(J1-Pad2)
- SW58 pad 1: Net-(D53-Pad2) -> Net-(J1-Pad3)
- SW59 pad 1: Net-(D54-Pad2) -> Net-(J1-Pad4)
- SW6 pad 1: Net-(D1-Pad2) -> Net-(J1-Pad1)
- SW60 pad 1: Net-(D55-Pad2) -> Net-(J1-Pad5)
- SW7 pad 1: Net-(D2-Pad2) -> Net-(J1-Pad2)
- SW8 pad 1: Net-(D3-Pad2) -> Net-(J1-Pad3)
- SW9 pad 1: Net-(D4-Pad2) -> Net-(J1-Pad4)

Commit message: Clean up, need to get switch clearances
Parts:
- moved D56 274.5 mm to (336.6, -132.1)
- moved D57 274.5 mm to (336.6, -127.0)
- moved D58 274.5 mm to (336.6, -120.7)
- moved D60 274.5 mm to (334.0, -110.5)
- moved D59 274.5 mm to (335.3, -115.6)
- moved D53 244.1 mm to (316.2, -120.7)
- moved D55 244.1 mm to (312.4, -110.5)
- moved D51 244.1 mm to (317.5, -129.5)
- moved D52 244.1 mm to (317.5, -124.5)
- moved D54 244.1 mm to (313.7, -115.6)
- moved D46 218.4 mm to (295.9, -130.8)
- moved D47 218.4 mm to (295.9, -125.7)
- moved D48 218.4 mm to (295.9, -120.7)
- moved D49 218.4 mm to (294.6, -115.6)
- moved D50 218.4 mm to (293.4, -111.8)
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
Commit message: Fix schematic, place components; need route
Parts:
- J2: moved to B.Cu
- moved J2 186.8 mm to (119.4, -3.81)
- moved D30 100.4 mm to (214.6, -12.7)
- moved D15 100.4 mm to (157.5, -12.7)
- moved D20 100.4 mm to (176.5, -12.7)
- moved D10 100.3 mm to (138.4, -12.7)
- moved D25 99.1 mm to (195.6, -12.7)
- moved D35 99.1 mm to (233.7, -12.7)
- moved D40 99.1 mm to (252.7, -12.7)
- moved D45 99.1 mm to (271.8, -12.7)
- moved D50 99.1 mm to (290.8, -12.7)
- moved D60 97.9 mm to (328.9, -12.7)
- moved D55 97.8 mm to (309.9, -12.7)
- moved D19 86.4 mm to (176.5, -31.8)
- moved D9 86.4 mm to (138.4, -31.8)
- moved D44 85.2 mm to (271.8, -31.8)
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Connections:
- SW41 pad 1: Net-(SW41-Pad1) -> Net-(J1-Pad1)
- SW42 pad 1: Net-(SW42-Pad1) -> Net-(J1-Pad2)
- SW43 pad 1: Net-(SW43-Pad1) -> Net-(J1-Pad3)
- SW44 pad 1: Net-(SW44-Pad1) -> Net-(J1-Pad4)
- SW45 pad 1: Net-(SW45-Pad1) -> Net-(J1-Pad5)
Routing:
- net Net-(J1-Pad5): track 0.00 -> 209.5 mm
- net Net-(J1-Pad4): track 0.00 -> 209.5 mm
- net Net-(J1-Pad3): track 0.00 -> 209.5 mm
- net Net-(J1-Pad2): track 0.00 -> 209.5 mm
- net Net-(J1-Pad1): track 0.00 -> 209.5 mm

Commit message: Fully routed, need to check layout
Parts:
- moved J2 8.89 mm to (119.4, 5.08)
Routing:
- net Net-(D56-Pad1): track 0.00 -> 265.2 mm
- net Net-(D51-Pad1): track 0.00 -> 249.9 mm
- net Net-(D46-Pad1): track 0.00 -> 232.9 mm
- net Net-(D41-Pad1): track 0.00 -> 215.6 mm
- net Net-(D36-Pad1): track 0.00 -> 199.1 mm
- net Net-(D31-Pad1): track 0.00 -> 182.6 mm
- net Net-(D26-Pad1): track 0.00 -> 166.1 mm
- net Net-(D21-Pad1): track 0.00 -> 149.6 mm
- net Net-(D16-Pad1): track 0.00 -> 133.1 mm
- net Net-(D11-Pad1): track 0.00 -> 116.6 mm
- net Net-(D1-Pad1): track 0.00 -> 102.9 mm
- net Net-(D10-Pad1): track 0.00 -> 100.8 mm
- net Net-(J1-Pad5): track 209.5 -> 283.5 mm
- net Net-(J1-Pad4): track 209.5 -> 267.0 mm
- net Net-(J1-Pad3): track 209.5 -> 254.7 mm
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
Commit message: Add generated gerbers
Parts:
- moved D1 160.1 mm to (36.8, 48.3)
- moved D10 160.1 mm to (55.9, 124.5)
- moved D11 160.1 mm to (74.9, 48.3)
- moved D12 160.1 mm to (74.9, 67.3)
- moved D13 160.1 mm to (74.9, 86.4)
- moved D14 160.1 mm to (74.9, 105.4)
- moved D15 160.1 mm to (74.9, 124.5)
- moved D16 160.1 mm to (94.0, 48.3)
- moved D17 160.1 mm to (94.0, 67.3)
- moved D18 160.1 mm to (94.0, 86.4)
- moved D19 160.1 mm to (94.0, 105.4)
- moved D2 160.1 mm to (36.8, 67.3)
- moved D20 160.1 mm to (94.0, 124.5)
- moved D21 160.1 mm to (113.0, 48.3)
- moved D22 160.1 mm to (113.0, 67.3)
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Other:
- board outline added: 251.5 x 128.3 mm
